File: Drone V3.kicad_sch (KiCad schematic)
At the start: 7 parts, among them J1 Supply, U5 STM32F427ZGTx

Commit message: MCU implementation start Still needs component schematic checks & component integration with MCU
Parts:
- added BOOT0_SW1: BOOT_Push, symbol Switch:SW_Push
- added C77, C80, C81, C82, C83, C84, C85, C86, C87, C88, C89, C90, C91, C92, C93, C94: 100n, symbol Device:C
- added C78, C79: 2.2u, symbol Device:C
- added NRST_SW1: NRST_Push, symbol Switch:SW_Push
- added R55: 20k, symbol Device:R
- added R56: 10k, symbol Device:R
Connections:
- net +3V3: now also U5.108 (VDD), U5.121 (VDD), U5.131 (VDD), U5.144 (VDD), U5.17 (VDD), U5.30 (VDD), U5.39 (VDD), U5.52 (VDD), U5.62 (VDD), U5.72 (VDD), U5.84 (VDD), U5.95 (VDD), BOOT0_SW1.1, C77.1, C80.1, C81.1, C82.1, C83.1, C84.1, C85.1, C86.1, C87.1, C88.1, C89.1, C90.1, C91.1, NRST_SW1.2
- net GND: now also U5.107 (VSS), U5.120 (VSS), U5.130 (VSS), U5.143 (PDR_ON), U5.16 (VSS), U5.31 (VSSA), U5.38 (VSS), U5.51 (VSS), U5.61 (VSS), U5.83 (VSS), U5.94 (VSS), C78.1, C79.1, C80.2, C81.2, C82.2, C83.2, C84.2, C85.2, C86.2, C87.2, C88.2, C89.2, C90.2, C91.2, C92.2, C93.2, C94.2, R55.1
- net NRST: now also U5.25 (NRST), C77.2, NRST_SW1.1
- net at U5.106 (VCAP_2): now also C79.2
- net at U5.138 (BOOT0): now also R56.2
- net VDDA: now reaches U5.32 (VREF+)
- net VDDA: now also U5.33 (VDDA), C92.1, C93.1, C94.1
- net at U5.71 (VCAP_1): now also C78.2
- new net: BOOT0_SW1.2, R55.2, R56.1
- no-connect marks 1 -> 2
Other:
- sheet Barometer ports: added +3.3V, Baro_DRI, Baro_SCL, Baro_SDA, GND; removed none
- sheet IMU1 ports: added +3.3V, GND, IMU_CS, IMU_FSYNC, IMU_INT1, IMU_INT2, IMU_SCLK, IMU_SDI, IMU_SDO; removed none
- sheet IMU2 ports: added +3.3V, GND, IMU_CS, IMU_FSYNC, IMU_INT1, IMU_INT2, IMU_SCLK, IMU_SDI, IMU_SDO; removed none
- sheet Mag1 ports: added +3.3V, GND, Mag_INT, Mag_SCL, Mag_SDA; removed none
- sheet Mag2 ports: added +3.3V, GND, Mag_INT, Mag_SCL, Mag_SDA; removed none
- sheet SDMicro ports: added +3.3V, GND, SD_CLK, SD_CS, SD_MISO, SD_MOSI; removed none
- sheet ToF ports: added +3.3V, GND, ToF_GPIO1, ToF_SCL, ToF_SDA, ToF_XSHUT, VDDA; removed none
- note added: "Altitude Sensing"
- note added: "Distance Sensor"
- note added: "GPS"
- note added: "MCU Decoupling"
- note added: "Pitch & Roll Sensing"
- note added: "Power Reg"
- note added: "SD-Micro"
- note added: "STM32F427ZGT"
- note added: "Transceiver"
- note added: "Yaw Sensing"
- moved on the sheet: U5

Commit message: Main Schematic update, Magnetometer deletions, Protocol connections, & External sensor compatibilities progress.
Parts:
- added J10, J13: SPI1, symbol Connector_Generic:Conn_01x04
- added J11: SPI2, symbol Connector_Generic:Conn_01x04
- added J12: SPI3, symbol Connector_Generic:Conn_01x04
- added J14: SPI5, symbol Connector_Generic:Conn_01x04
- added J15: SPI6, symbol Connector_Generic:Conn_01x04
- added J16: I2C1, symbol Connector_Generic:Conn_01x02
- added J17: I2C2, symbol Connector_Generic:Conn_01x02
- added J18: I2C3, symbol Connector_Generic:Conn_01x02
- added J19: CAN1, symbol Connector_Generic:Conn_01x02
- added J2: USART1, symbol Connector_Generic:Conn_01x05
- added J20: CAN2, symbol Connector_Generic:Conn_01x02
- added J21: Supplies, symbol Connector_Generic:Conn_02x24_Counter_Clockwise
- added J22: Grounds, symbol Connector_Generic:Conn_01x24
- added J5: USART2, symbol Connector_Generic:Conn_01x05
- added J6: USART3, symbol Connector_Generic:Conn_01x05
- added J7, J8: UART4, symbol Connector_Generic:Conn_01x02
- added J9: USART6, symbol Connector_Generic:Conn_01x05
Connections:
- net +3V3: now also J21.1 (Pin_1), J21.10 (Pin_10), J21.11 (Pin_11), J21.12 (Pin_12), J21.13 (Pin_13), J21.14 (Pin_14), J21.15 (Pin_15), J21.16 (Pin_16), J21.17 (Pin_17), J21.18 (Pin_18), J21.19 (Pin_19), J21.2 (Pin_2), J21.20 (Pin_20), J21.21 (Pin_21), J21.22 (Pin_22), J21.23 (Pin_23), J21.24 (Pin_24), J21.3 (Pin_3), J21.4 (Pin_4), J21.5 (Pin_5), J21.6 (Pin_6), J21.7 (Pin_7), J21.8 (Pin_8), J21.9 (Pin_9)
- net +5V: now also J21.25 (Pin_25), J21.26 (Pin_26), J21.27 (Pin_27), J21.28 (Pin_28), J21.29 (Pin_29), J21.30 (Pin_30), J21.31 (Pin_31), J21.32 (Pin_32), J21.33 (Pin_33), J21.34 (Pin_34), J21.35 (Pin_35), J21.36 (Pin_36), J21.37 (Pin_37), J21.38 (Pin_38), J21.39 (Pin_39), J21.40 (Pin_40), J21.41 (Pin_41), J21.42 (Pin_42), J21.43 (Pin_43), J21.44 (Pin_44), J21.45 (Pin_45), J21.46 (Pin_46), J21.47 (Pin_47), J21.48 (Pin_48)
- net GND: now also J22.1 (Pin_1), J22.10 (Pin_10), J22.11 (Pin_11), J22.12 (Pin_12), J22.13 (Pin_13), J22.14 (Pin_14), J22.15 (Pin_15), J22.16 (Pin_16), J22.17 (Pin_17), J22.18 (Pin_18), J22.19 (Pin_19), J22.2 (Pin_2), J22.20 (Pin_20), J22.21 (Pin_21), J22.22 (Pin_22), J22.23 (Pin_23), J22.24 (Pin_24), J22.3 (Pin_3), J22.4 (Pin_4), J22.5 (Pin_5), J22.6 (Pin_6), J22.7 (Pin_7), J22.8 (Pin_8), J22.9 (Pin_9)
- net GPS_RX: now also U5.113 (PC12), J8.2 (Pin_2)
- net GPS_TX: now also U5.116 (PD2), J8.1 (Pin_1)
- net IMU_MISO: now also U5.42 (PA6)
- net IMU_MOSI: now also U5.43 (PA7)
- net SD_MISO: now also U5.134 (PB4)
- net SD_MOSI: now also U5.135 (PB5)
- net TSVR_RX: now also U5.34 (PA0)
- net TSVR_TX: now also U5.35 (PA1)
- net USART1_CK: now reaches U5.100 (PA8)
- net USART1_CK: now also J2.5 (Pin_5)
- net USART1_TX: now reaches U5.101 (PA9)
- net USART1_TX: now also J2.4 (Pin_4)
- net USART1_RX: now reaches U5.102 (PA10)
- net USART1_RX: now also J2.3 (Pin_3)
- net USART1_CTS: now reaches U5.103 (PA11)
- net USART1_CTS: now also J2.2 (Pin_2)
- net USART1_RTS: now reaches U5.104 (PA12)
- net USART1_RTS: now also J2.1 (Pin_1)
- net USART2_CTS: now reaches U5.117 (PD3)
- net USART2_CTS: now also J5.2 (Pin_2)
- net USART2_RTS: now reaches U5.118 (PD4)
- net USART2_RTS: now also J5.1 (Pin_1)
- net USART2_TX: now reaches U5.119 (PD5)
- net USART2_TX: now also J5.4 (Pin_4)
- net USART2_RX: now reaches U5.122 (PD6)
- net USART2_RX: now also J5.3 (Pin_3)
- net USART2_CK: now reaches U5.123 (PD7)
- net USART2_CK: now also J5.5 (Pin_5)
- net USART6_RX: now reaches U5.124 (PG9)
- net USART6_RX: now also J9.3 (Pin_3)
- net USART6_CTS: now reaches U5.128 (PG13)
- net USART6_CTS: now also J9.2 (Pin_2)
- net USART6_TX: now reaches U5.129 (PG14)
- net USART6_TX: now also J9.4 (Pin_4)
- net SD_SCK: now reaches U5.133 (PB3)
- net Sense_SCL: now reaches U5.136 (PB6)
- net Sense_SDA: now reaches U5.137 (PB7)
- net OpF_MISO: now reaches U5.28 (PC2)
- net OpF_MOSI: now reaches U5.29 (PC3)
- net IMU_SCK: now reaches U5.41 (PA5)
- net OpF_SCK: now reaches U5.74 (PB13)
- net USART3_TX: now reaches U5.77 (PD8)
- net USART3_TX: now also J6.4 (Pin_4)
- net USART3_RX: now reaches U5.78 (PD9)
- net USART3_RX: now also J6.3 (Pin_3)
- net USART3_CK: now reaches U5.79 (PD10)
- net USART3_CK: now also J6.5 (Pin_5)
- net USART3_CTS: now reaches U5.80 (PD11)
- net USART3_CTS: now also J6.2 (Pin_2)
- net USART3_RTS: now reaches U5.81 (PD12)
- net USART3_RTS: now also J6.1 (Pin_1)
- net USART6_CK: now reaches U5.92 (PG7)
- net USART6_CK: now also J9.5 (Pin_5)
- net USART6_RTS: now reaches U5.93 (PG8)
- net USART6_RTS: now also J9.1 (Pin_1)
- new net CAN1_RX: J19.1 (Pin_1)
- new net CAN1_TX: J19.2 (Pin_2)
- new net CAN2_RX: J20.1 (Pin_1)
- new net CAN2_TX: J20.2 (Pin_2)
- new net I2C1_SCL: J16.2 (Pin_2)
- new net I2C1_SDA: J16.1 (Pin_1)
- new net I2C2_SCL: J17.2 (Pin_2)
- new net I2C2_SDA: J17.1 (Pin_1)
- new net I2C3_SCL: J18.2 (Pin_2)
- new net I2C3_SDA: J18.1 (Pin_1)
- new net SPI1_CS: J10.4 (Pin_4)
- new net SPI1_MISO: J10.2 (Pin_2)
- new net SPI1_MOSI: J10.1 (Pin_1)
- new net SPI1_SCK: J10.3 (Pin_3)
- new net SPI2_CS: J11.4 (Pin_4)
- new net SPI2_MISO: J11.2 (Pin_2)
- new net SPI2_MOSI: J11.1 (Pin_1)
- new net SPI2_SCK: J11.3 (Pin_3)
- new net SPI3_CS: J12.4 (Pin_4)
- new net SPI3_MISO: J12.2 (Pin_2)
- new net SPI3_MOSI: J12.1 (Pin_1)
- new net SPI3_SCK: J12.3 (Pin_3)
- new net SPI4_CS: J13.4 (Pin_4)
- new net SPI4_MISO: J13.2 (Pin_2)
- new net SPI4_MOSI: J13.1 (Pin_1)
- new net SPI4_SCK: J13.3 (Pin_3)
- new net SPI5_CS: J14.4 (Pin_4)
- new net SPI5_MISO: J14.2 (Pin_2)
- new net SPI5_MOSI: J14.1 (Pin_1)
- new net SPI5_SCK: J14.3 (Pin_3)
- new net SPI6_CS: J15.4 (Pin_4)
- new net SPI6_MISO: J15.2 (Pin_2)
- new net SPI6_MOSI: J15.1 (Pin_1)
- new net SPI6_SCK: J15.3 (Pin_3)
- new net UART4_RX: J7.1 (Pin_1)
- new net UART4_TX: J7.2 (Pin_2)
- no-connect marks 2 -> 6
Other:
- removed sheet Mag1
- removed sheet Mag2
- added sheet OpticalFlow (opticalflow.kicad_sch)
- note added: "I2C1_SCL"
- note added: "I2C1_SDA"
- note added: "Optical Flow"
- note added: "Protocol Ports"
- note added: "SPI1_MISO"
- note added: "SPI1_MOSI"
- note added: "SPI1_SCK"
- note added: "SPI2_MISO"
- note added: "SPI2_MOSI"
- note added: "SPI2_SCK"
- note added: "SPI3_MISO"
- note added: "SPI3_MOSI"
- note added: "SPI3_SCK"
- note added: "Sensor Supplies"
- note added: "UART4_RX"
- note added: "UART4_TX"
- note added: "UART5_RX"
- note added: "UART5_TX"
- note removed: "Yaw Sensing"
- moved on the sheet: G1, G2

Commit message: MCU Integration & Sensor Ports
Parts:
- removed J2: USART1, symbol Connector_Generic:Conn_01x05
- removed J5: USART2, symbol Connector_Generic:Conn_01x05
- removed J6: USART3, symbol Connector_Generic:Conn_01x05
- removed J9: USART6, symbol Connector_Generic:Conn_01x05
- added C98, C99: 22p, symbol Device:C
- added D18: MCU_LED1, symbol Device:LED
- added D19: MCU_LED2, symbol Device:LED
- added D20: SD_LED, symbol Device:LED
- added J2: USART1, symbol Connector_Generic:Conn_01x02
- added J23: UART7, symbol Connector_Generic:Conn_01x02
- added J24: UART8, symbol Connector_Generic:Conn_01x02
- added J25: GPIO, symbol Connector_Generic:Conn_02x24_Counter_Clockwise
- added J5: USART2, symbol Connector_Generic:Conn_01x02
- added J6: USART3, symbol Connector_Generic:Conn_01x02
- added J9: USART6, symbol Connector_Generic:Conn_01x02
- added R39, R57, R58: 220, symbol Device:R
- added R40, R41, R42, R43, R44, R45: 1.8k, symbol Device:R
- added R49, R5, R51, R53, R54, R59, R60: 10k, symbol Device:R
- added Y1: 16MHz, symbol Device:Crystal
- J8: value UART4 -> UART5
Connections:
- net OpF_SCK is gone; now on net CAN2_TX: U5.74 (PB13)
- net SPI1_MISO is gone; now on net SPI1_MISO_IMU: J10.2 (Pin_2)
- net SPI1_MOSI is gone; now on net SPI1_MOSI_IMU: J10.1 (Pin_1)
- net SPI1_SCK is gone; now on net SPI1_SCK_IMU: J10.3 (Pin_3)
- net SPI2_MISO is gone; now on net SPI2_MISO_OpF: J11.2 (Pin_2)
- net SPI2_MOSI is gone; now on net SPI2_MOSI_OpF: J11.1 (Pin_1)
- net SPI3_MISO is gone; now on net SPI3_MISO_SD: J12.2 (Pin_2)
- net SPI3_MOSI is gone; now on net SPI3_MOSI_SD: J12.1 (Pin_1)
- net SPI3_SCK is gone; now on net SPI3_SCK_SD: J12.3 (Pin_3)
- net Sense_SCL is gone; now on net I2C1_SCL_Sense: U5.136 (PB6)
- net Sense_SDA is gone; now on net I2C1_SDA_Sense: U5.137 (PB7)
- net UART4_RX is gone; now on net UART4_RX_TSVR: J7.1 (Pin_1)
- net UART4_TX is gone; now on net UART4_TX_TSVR: J7.2 (Pin_2)
- net USART1_CK is gone; now on net I2C3_SCL: U5.100 (PA8)
- net USART1_CTS is gone; now on net IMU1_CS: U5.103 (PA11)
- net USART1_RTS is gone; now on net IMU2_CS: U5.104 (PA12)
- net USART2_CTS is gone; now on net SPI2_SCK_OpF: U5.117 (PD3)
- net USART2_RTS is gone; now on net OpF_LDO_EN: U5.118 (PD4)
- net USART6_CTS is gone; now on net SPI6_SCK: U5.128 (PG13)
- net +3V3: now also R40.1, R41.1, R42.1, R43.1, R44.1, R45.1, R49.1, R51.1, R53.1, R54.1, R59.1, R60.1
- net 12VBuckEN: now also U5.7 (PC13)
- net CAN1_RX: now also U5.114 (PD0)
- net CAN1_TX: now also U5.115 (PD1)
- net CAN2_RX: now also U5.73 (PB12)
- net I2C2_SCL: now also U5.11 (PF1), R43.2
- net I2C2_SDA: now also U5.10 (PF0), R42.2
- net I2C3_SCL: now also R45.2
- net I2C3_SDA: now also U5.99 (PC9), R44.2
- net IMU1_INT1: now also U5.139 (PB8)
- net IMU2_INT2: now also U5.140 (PB9)
- net OpF_MOTION: now also U5.112 (PC11)
- net OpF_NCS: now also U5.111 (PC10)
- net OpF_NRESET: now also U5.98 (PC8), R5.2
- net SD_CS: now also U5.48 (PB2)
- net SPI1_CS: now also U5.56 (PG0)
- net SPI2_CS: now also U5.57 (PG1)
- net SPI3_CS: now also U5.87 (PG2)
- net SPI4_CS: now also U5.88 (PG3)
- net SPI4_MISO: now also U5.4 (PE5), R54.2
- net SPI4_MOSI: now also U5.5 (PE6)
- net SPI4_SCK: now also U5.1 (PE2)
- net SPI5_CS: now also U5.89 (PG4)
- net SPI5_MISO: now also U5.20 (PF8), R59.2
- net SPI5_MOSI: now also U5.21 (PF9)
- net SPI5_SCK: now also U5.19 (PF7)
- net SPI6_CS: now also U5.90 (PG5)
- net SPI6_MISO: now also U5.127 (PG12), R60.2
- net SPI6_MOSI: now also U5.129 (PG14)
- net SWCLK: now also U5.109 (PA14)
- net SWDIO: now also U5.105 (PA13)
- net USART1_RX: now also J2.1 (Pin_1)
- net USART1_TX: now also J2.2 (Pin_2)
- net USART2_RX: now also J5.1 (Pin_1)
- net USART2_TX: now also J5.2 (Pin_2)
- net USART3_RX: now also J6.1 (Pin_1)
- net USART3_TX: now also J6.2 (Pin_2)
- net USART6_RX: now also U5.97 (PC7), J9.1 (Pin_1); no longer U5.124 (PG9)
- net USART6_TX: now also U5.96 (PC6), J9.2 (Pin_2); no longer U5.129 (PG14)
- net VSense: now also U5.45 (PC5)
- net IMU_FSYNC: now reaches U5.110 (PA15)
- net PF2_D: now reaches U5.12 (PF2)
- net PF2_D: now also J25.18 (Pin_18)
- net PG10_D: now reaches U5.125 (PG10)
- net PG10_D: now also J25.45 (Pin_45)
- net PG11_D: now reaches U5.126 (PG11)
- net PG11_D: now also J25.44 (Pin_44)
- net PF3_A: now reaches U5.13 (PF3)
- net PF3_A: now also J25.32 (Pin_32)
- net PG15_D: now reaches U5.132 (PG15)
- net PG15_D: now also J25.43 (Pin_43)
- net PF4_A: now reaches U5.14 (PF4)
- net PF4_A: now also J25.31 (Pin_31)
- net UART8_RX: now reaches U5.141 (PE0)
- net UART8_RX: now also J24.1 (Pin_1)
- net UART8_TX: now reaches U5.142 (PE1)
- net UART8_TX: now also J24.2 (Pin_2)
- net PF5_A: now reaches U5.15 (PF5)
- net PF5_A: now also J25.30 (Pin_30)
- net PF6_A: now reaches U5.18 (PF6)
- net PF6_A: now also J25.29 (Pin_29)
- net PE3_D: now reaches U5.2 (PE3)
- net PE3_D: now also J25.9 (Pin_9)
- net PF10_A: now reaches U5.22 (PF10)
- net PF10_A: now also J25.28 (Pin_28)
- net at U5.23 (PH0): now also C98.2
- net at U5.24 (PH1): now also C99.1
- net PC0_A: now reaches U5.26 (PC0)
- net PC0_A: now also J25.37 (Pin_37)
- net PC1_A: now reaches U5.27 (PC1)
- net PC1_A: now also J25.36 (Pin_36)
- net PE4_D: now reaches U5.3 (PE4)
- net PA2_A: now reaches U5.36 (PA2)
- net PA2_A: now also J25.42 (Pin_42)
- net PA3_A: now reaches U5.37 (PA3)
- net PA3_A: now also J25.41 (Pin_41)
- net PA4_A: now reaches U5.40 (PA4)
- net PA4_A: now also J25.40 (Pin_40)
- net PC4_A: now reaches U5.44 (PC4)
- net PC4_A: now also J25.33 (Pin_33)
- net PB0_A: now reaches U5.46 (PB0)
- net PB0_A: now also J25.39 (Pin_39)
- net PB1_A: now reaches U5.47 (PB1)
- net PB1_A: now also J25.38 (Pin_38)
- net PF11_D: now reaches U5.49 (PF11)
- net PF11_D: now also J25.19 (Pin_19)
- net PF12_D: now reaches U5.50 (PF12)
- net PF12_D: now also J25.20 (Pin_20)
- net PF13_D: now reaches U5.53 (PF13)
- net PF13_D: now also J25.21 (Pin_21)
- net PF14_D: now reaches U5.54 (PF14)
- net PF14_D: now also J25.22 (Pin_22)
- net UART7_RX: now reaches U5.58 (PE7)
- net UART7_RX: now also J23.1 (Pin_1)
- net UART7_TX: now reaches U5.59 (PE8)
- net UART7_TX: now also J23.2 (Pin_2)
- net PE9_D: now reaches U5.60 (PE9)
- net PE9_D: now also J25.11 (Pin_11)
- net PE10_D: now reaches U5.63 (PE10)
- net PE10_D: now also J25.12 (Pin_12)
- net PE11_D: now reaches U5.64 (PE11)
- net PE11_D: now also J25.13 (Pin_13)
- net PE12_D: now reaches U5.65 (PE12)
- net PE12_D: now also J25.14 (Pin_14)
- net PE13_D: now reaches U5.66 (PE13)
- net PE13_D: now also J25.15 (Pin_15)
- net PE14_D: now reaches U5.67 (PE14)
- net PE14_D: now also J25.16 (Pin_16)
- net MCU_LED1: now reaches U5.69 (PB10)
- net MCU_LED1: now also D18.1 (K)
- net MCU_LED2: now reaches U5.70 (PB11)
- net MCU_LED2: now also D19.1 (K)
- net SPI2_MISO_OpF: now reaches U5.75 (PB14)
- net SPI2_MISO_OpF: now also R51.2
- net SPI2_MOSI_OpF: now reaches U5.76 (PB15)
- net SD_LED: now reaches U5.8 (PC14)
- net SD_LED: now also D20.1 (K)
- net PD13_D: now reaches U5.82 (PD13)
- net PD13_D: now also J25.6 (Pin_6)
- net PD14_D: now reaches U5.85 (PD14)
- net PD14_D: now also J25.7 (Pin_7)
- net PC15_D: now reaches U5.9 (PC15)
- net PC15_D: now also J25.1 (Pin_1)
- net PG6_D: now reaches U5.91 (PG6)
- net PG6_D: now also J25.24 (Pin_24)
- net GPS_RX renamed UART5_TX_GPS
- net GPS_TX renamed UART5_RX_GPS
- net I2C1_SCL renamed I2C1_SCL_Sense
- net I2C1_SCL_Sense: now also R41.2
- net I2C1_SDA renamed I2C1_SDA_Sense
- net I2C1_SDA_Sense: now also R40.2
- net IMU_MISO renamed SPI1_MISO_IMU
- net SPI1_MISO_IMU: now also R49.2
- net IMU_MOSI renamed SPI1_MOSI_IMU
- net IMU_SCK renamed SPI1_SCK_IMU
- net OpF_MISO renamed PC2_A
- net PC2_A: now also J25.35 (Pin_35)
- net OpF_MOSI renamed PC3_A
- net PC3_A: now also J25.34 (Pin_34)
- net SD_MISO renamed SPI3_MISO_SD
- net SPI3_MISO_SD: now also R53.2
- net SD_MOSI renamed SPI3_MOSI_SD
- net SD_SCK renamed SPI3_SCK_SD
- net SPI2_SCK renamed SPI2_SCK_OpF
- net TSVR_RX renamed UART4_TX_TSVR
- net TSVR_TX renamed UART4_RX_TSVR
- net USART2_CK renamed PD7_D
- net PD7_D: now also J25.2 (Pin_2)
- net USART3_CK renamed PD10_D
- net PD10_D: now also J25.3 (Pin_3)
- net USART3_CTS renamed PD11_D
- net PD11_D: now also J25.4 (Pin_4)
- net USART3_RTS renamed PD12_D
- net PD12_D: now also J25.5 (Pin_5)
- net USART6_CK renamed PG7_D
- net PG7_D: now also J25.48 (Pin_48)
- net USART6_RTS renamed PG8_D
- net PG8_D: now also J25.47 (Pin_47)
- new net: C98.1, Y1.1
- new net: C99.2, Y1.2
- new net: D19.2 (A), R57.1
- new net: D18.2 (A), R39.1
- new net: D20.2 (A), R58.1
- new net +3.3V: R39.2, R5.1, R57.2, R58.2
- new net PG9_D: J25.46 (Pin_46), U5.124 (PG9)
- no-connect marks 6 -> 8
Other:
- sheet GPS ports: added none; removed GPS_SCL, GPS_SDA
- note added: "ADC123_IN10"
- note added: "ADC123_IN11"
- note added: "ADC123_IN12"
- note added: "ADC123_IN13"
- note added: "ADC123_IN2"
- note added: "ADC123_IN3"
- note added: "ADC12_IN14"
- note added: "ADC12_IN15"
- note added: "ADC12_IN4"
- note added: "ADC12_IN8"
- note added: "ADC12_IN9"
- note added: "ADC3_IN14"
- note added: "ADC3_IN15"
- note added: "ADC3_IN4"
- note added: "ADC3_IN8"
- note added: "ADC3_IN9"
- note added: "Analog: A2-A4"
- note added: "Analog: B0 & B1"
- note added: "CAN1_RX"
- note added: "CAN1_TX"
- note added: "CAN2_RX"
- note added: "CAN2_TX"
- note added: "Debug LED1"
- note added: "Debug LED2"
- note added: "Debug LEDs"
- note added: "GPIO Pins"
- note added: "I2C2_SCL"
- note added: "I2C2_SDA"
- note added: "I2C3_SCL"
- note added: "I2C3_SDA"
- note added: "IO: C15 Analog: PC0-4"
- note added: "IO: D7, & D10-D15"
- note added: "IO: E3, E4, & E9-E15"
- note added: "IO: F2 & F11-F15 Analog: F3-F6 & F10"
- note added: "IO: G6-G11 & G15"
- note added: "JTCK-SWCLK"
- note added: "JTMS-SWDIO"
- note added: "SDMicro LED"
- note added: "SPI4_MISO"
- note added: "SPI4_MOSI"
- note added: "SPI4_SCK"
- note added: "SPI5_MISO"
- note added: "SPI5_MOSI"
- note added: "SPI5_SCK"
- note added: "SPI6_MISO"
- note added: "SPI6_MOSI"
- note added: "SPI6_SCK"
- note added: "TIM2_CH1"
- note added: "UART7_RX"
- note added: "UART7_TX"
- note added: "UART8_RX"
- note added: "UART8_TX"
- note added: "USART1_RX"
- note added: "USART1_TX"
- note added: "USART2_RX"
- note added: "USART2_TX"
- note added: "USART3_RX"
- note added: "USART3_TX"
- note added: "USART6_RX"
- note added: "USART6_TX"
- moved on the sheet: C77, C78, C79, J10, J11, J12, J13, J14, J15, J16, J17, J18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

Commit message: USB C integration, 5V tolerances on UART ports, digital pins, and analog pins.
Parts:
- added C100, C101, C102, C103, C104, C105: 100n, symbol Device:C
- added D21: ESD CLAMP, Library:SOT-563_L1.6-W1.2-P0.50-LS1.6-BL, symbol Library:USBLC6-2P6_C49451919
- added R46, R64, R68, R72: 1.7k, symbol Device:R
- added R50, R65, R69, R73: 3.3k, symbol Device:R
- added R52, R61, R62, R63, R66, R67, R70, R71: 0, symbol Device:R
- added R74, R75: 5.1k, symbol Device:R
- added TXB0, TXB1, TXB2: TXB0104RUT, Package_DFN_QFN:Texas_R-PUQFN-N12, symbol Logic_LevelTranslator:TXB0104RUT
- added U16: USBC, Library:USB-C-SMD_G-SWITCH_GT-USB-7010ASV, symbol Library:GT-USB-7010ASV
Connections:
- net +3V3: now also C100.2, C102.2, C104.2, TXB0.1 (VCCA), TXB0.12 (OE), TXB1.1 (VCCA), TXB1.12 (OE), TXB2.1 (VCCA), TXB2.12 (OE)
- net +5V: now also C101.2, C103.2, C105.2, D21.5 (VBUS), TXB0.11 (VCCB), TXB1.11 (VCCB), TXB2.11 (VCCB), U16.A4B9 (VBUS), U16.B4A9 (VBUS)
- net GND: now also C100.1, C101.1, C102.1, C103.1, C104.1, C105.1, D21.2 (GND), R50.2, R65.2, R69.2, R73.2, R74.2, R75.2, TXB0.6 (GND), TXB1.6 (GND), TXB2.6 (GND), U16.1 (SHELL), U16.2 (SHELL), U16.3 (SHELL), U16.4 (SHELL), U16.A1B12 (GND), U16.B1A12 (GND)
- net IMU1_CS: now also U5.91 (PG6); no longer U5.103 (PA11)
- net IMU1_INT1: now also U5.93 (PG8); no longer U5.139 (PB8)
- net IMU2_CS: now also U5.92 (PG7); no longer U5.104 (PA12)
- net IMU2_INT2: now also U5.124 (PG9); no longer U5.140 (PB9)
- net PA2_A: now also R52.1, R61.2; no longer J25.42 (Pin_42)
- net PA3_A: now also R62.1, R63.2; no longer J25.41 (Pin_41)
- net PA4_A: now also R66.1, R67.2; no longer J25.40 (Pin_40)
- net PB0_A: now also R70.1, R71.2; no longer J25.39 (Pin_39)
- net PB1_A: now also J25.42 (Pin_42); no longer J25.38 (Pin_38)
- net PC0_A: now also J25.41 (Pin_41); no longer J25.37 (Pin_37)
- net PC15_D: now also TXB2.2 (A1); no longer J25.1 (Pin_1)
- net PC1_A: now also J25.40 (Pin_40); no longer J25.36 (Pin_36)
- net PC2_A: now also J25.39 (Pin_39); no longer J25.35 (Pin_35)
- net PC3_A: now also J25.38 (Pin_38); no longer J25.34 (Pin_34)
- net PC4_A: now also J25.37 (Pin_37); no longer J25.33 (Pin_33)
- net PD10_D: now also TXB2.4 (A3); no longer J25.3 (Pin_3)
- net PD11_D: now also TXB2.5 (A4); no longer J25.4 (Pin_4)
- net PD7_D: now also TXB2.3 (A2); no longer J25.2 (Pin_2)
- net PF10_A: now also J25.32 (Pin_32); no longer J25.28 (Pin_28)
- net PF3_A: now also J25.36 (Pin_36); no longer J25.32 (Pin_32)
- net PF4_A: now also J25.35 (Pin_35); no longer J25.31 (Pin_31)
- net PF5_A: now also J25.34 (Pin_34); no longer J25.30 (Pin_30)
- net PF6_A: now also J25.33 (Pin_33); no longer J25.29 (Pin_29)
- net PG10_D: now also J25.24 (Pin_24); no longer J25.45 (Pin_45)
- net PG11_D: now also J25.48 (Pin_48); no longer J25.44 (Pin_44)
- net PG15_D: now also J25.47 (Pin_47); no longer J25.43 (Pin_43)
- net Servo1: now also U5.139 (PB8)
- net Servo2: now also U5.140 (PB9)
- net UART7_RX: now also TXB1.3 (A2); no longer J23.1 (Pin_1)
- net UART7_TX: now also TXB1.2 (A1); no longer J23.2 (Pin_2)
- net UART8_RX: now also TXB1.5 (A4); no longer J24.1 (Pin_1)
- net UART8_TX: now also TXB1.4 (A3); no longer J24.2 (Pin_2)
- net USART3_RX: now also TXB0.3 (A2); no longer J6.1 (Pin_1)
- net USART3_TX: now also TXB0.2 (A1); no longer J6.2 (Pin_2)
- net USART6_RX: now also TXB0.5 (A4); no longer J9.1 (Pin_1)
- net USART6_TX: now also TXB0.4 (A3); no longer J9.2 (Pin_2)
- removed net PG6_D: J25.24 (Pin_24), U5.91 (PG6)
- removed net PG7_D: J25.48 (Pin_48), U5.92 (PG7)
- removed net PG8_D: J25.47 (Pin_47), U5.93 (PG8)
- net PG9_D renamed PA2_A_5V
- net PA2_A_5V: now also R46.1, R61.1; no longer U5.124 (PG9)
- new net: R70.2, R72.2, R73.1
- new net: R62.2, R64.2, R65.1
- new net: R66.2, R68.2, R69.1
- new net: R46.2, R50.1, R52.2
- new net: R75.1, U16.A5 (CC1)
- new net: D21.1 (I/O1), U16.A6 (DP1), U16.B6 (DP2)
- new net: D21.3 (I/O2), U16.A7 (DN1), U16.B7 (DN2)
- new net: R74.1, U16.B5 (CC2)
- new net OTG_FS_DM: D21.4 (I/O2), U5.103 (PA11)
- new net OTG_FS_DP: D21.6 (I/O1), U5.104 (PA12)
- new net PA3_A_5V: J25.45 (Pin_45), R63.1, R64.1
- new net PA4_A_5V: J25.44 (Pin_44), R67.1, R68.1
- new net PB0_A_5V: J25.43 (Pin_43), R71.1, R72.1
- new net PC15_D_5V: J25.1 (Pin_1), TXB2.10 (B1)
- new net PD10_D_5V: J25.3 (Pin_3), TXB2.8 (B3)
- new net PD11_D_5V: J25.4 (Pin_4), TXB2.7 (B4)
- new net PD7_D_5V: J25.2 (Pin_2), TXB2.9 (B2)
- new net UART7_RX_5V: J23.1 (Pin_1), TXB1.9 (B2)
- new net UART7_TX_5V: J23.2 (Pin_2), TXB1.10 (B1)
- new net UART8_RX_5V: J24.1 (Pin_1), TXB1.7 (B4)
- new net UART8_TX_5V: J24.2 (Pin_2), TXB1.8 (B3)
- new net USART3_RX_5V: J6.1 (Pin_1), TXB0.9 (B2)
- new net USART3_TX_5V: J6.2 (Pin_2), TXB0.10 (B1)
- new net USART6_RX_5V: J9.1 (Pin_1), TXB0.7 (B4)
- new net USART6_TX_5V: J9.2 (Pin_2), TXB0.8 (B3)
- no-connect marks 8 -> 14
Other:
- note added: "5V PA2 Sensor: Bridge R52 & Disconnect R61 3.3V PA2 Sensor: Bridge R61 & Disconnect R52 1 of the 2 resistors should be bridged at a time."
- note added: "5V Sensor Tolerance"
- note added: "USB-C Port"
