File: esc1.kicad_sch (KiCad schematic)
At the start: 86 parts, among them J2 Phase Outputs, J3 Pad Terminals, J4 Signal, U1 IRS21867S, U13 STM32F303CBTx, U4 INA180A3, U6 IRS21867S, U7 IRS21867S, U9 INA180A3

Commit message: ESC PCB Finalized Iteration #1
Parts:
- added R14: 0, easyeda2kicad:R0805, symbol Device:R
Connections:
- net +ESC: now also 12V_SD1.4 (EN), 12V_SD1.5 (VIN), C42.1
- net -3V3MCU: now also R14.1; no longer U13.8 (VSSA)
- new net VSSA: R14.2, U13.8 (VSSA)

Commit message: Sensors & Main board start
Parts:
- removed 12V_SD1: TPS560430, easyeda2kicad:SOT-23-6_L2.9-W1.6-P0.95-LS2.8-BL, symbol easyeda2kicad:TPS560430XDBVR
- removed C21, C23, C24: 1u, Capacitor_SMD:C_0805_2012Metric, symbol Device:C
- removed C29: 100n, easyeda2kicad:C0805, symbol Device:C
- removed C40: 22n, Capacitor_SMD:C_0805_2012Metric, symbol Device:C
- removed C42: 2.2u, Capacitor_SMD:C_0805_2012Metric, symbol Device:C
- removed C43: 100n, Capacitor_SMD:C_0805_2012Metric, symbol Device:C
- removed C45: 10u, Capacitor_SMD:C_0805_2012Metric, symbol Device:C
- removed J2: Phase Outputs, CustomFPs:ESC Outputs, symbol Connector_Generic:Conn_01x03
- removed L6: 33u, easyeda2kicad:IND-SMD_L3.0-W3.0_LQH3NPN2R2NG0L, symbol Device:L
- removed R39: 243, easyeda2kicad:R0805, symbol Device:R
- removed R40: 22.1, easyeda2kicad:R0805, symbol Device:R
- added 12V_SD1: XL1509-12, Package_SO:SOIC-8_3.9x4.9mm_P1.27mm, symbol Regulator_Switching:XL1509-12
- added C17, C50: 100n, symbol Device:C
- added C18, C51: 1n, symbol Device:C
- added C21, C29, C42: 1u, symbol Device:C_Polarized
- added C43: 470u, symbol Device:C_US
- added C44: 1u, symbol Device:C
- added C45: 180u, symbol Device:C_US
- added D11, D13, D9: SMBJ33A, PCM_JLCPCB:D_SMB, symbol PCM_JLCPCB-Diodes:TVS-Uni,SMBJ33A
- added D16: 1N5820, Diode_THT:D_DO-201AD_P15.24mm_Horizontal, symbol Diode:1N5820
- added L5: 68u, symbol Device:L
- added R15: 1k, symbol Device:R
- added U8: INA180A3, Package_TO_SOT_SMD:SOT-23-5, symbol Amplifier_Current:INA180A3
- BOOT0_SW: renamed from BOOT0_SW1; footprint easyeda2kicad:SW-SMD_4P-L3.5-W3.0-P1.50-LS4.7 -> (none)
- C15, C20, C26, C28, C33, C34, C35, C37, C39: footprint easyeda2kicad:C0805 -> (none)
- C16, C22, C31, C32, C36, C38, C41: footprint Capacitor_SMD:C_0805_2012Metric -> (none)
- C19, C25, C49: value 22n -> 100n; footprint Capacitor_SMD:C_0805_2012Metric -> (none)
- C27: value 22n -> 1n; footprint Capacitor_SMD:C_0805_2012Metric -> (none)
- C30: footprint easyeda2kicad:CAP-TH_BD12.5-P5.00-D0.6-FD -> (none)
- D10, D12, D8: footprint easyeda2kicad:SOD-323_L1.8-W1.3-LS2.5-RD -> Diode_SMD:D_SOD-323
- D14, D15, D17: footprint LED_SMD:LED_0805_2012Metric -> (none)
- J3: footprint CustomFPs:Battery Inputs -> Library:VCC Pads
- J4: footprint Connector_PinHeader_2.54mm:PinHeader_1x03_P2.54mm_Horizontal -> (none)
- NRST_SW: renamed from NRST_SW1; footprint easyeda2kicad:SW-SMD_4P-L3.5-W3.0-P1.50-LS4.7 -> (none)
- Q1: renamed from NMOS1; footprint easyeda2kicad:DFN-8_L5.9-W5.2-P1.27-LS6.2-BL -> (none)
- Q2: renamed from NMOS2; footprint easyeda2kicad:DFN-8_L5.9-W5.2-P1.27-LS6.2-BL -> (none)
- Q3: renamed from NMOS3; footprint easyeda2kicad:DFN-8_L5.9-W5.2-P1.27-LS6.2-BL -> (none)
- Q4: renamed from NMOS4; footprint easyeda2kicad:DFN-8_L5.9-W5.2-P1.27-LS6.2-BL -> (none)
- Q5: renamed from NMOS5; footprint easyeda2kicad:DFN-8_L5.9-W5.2-P1.27-LS6.2-BL -> (none)
- Q6: renamed from NMOS6; value HYG025N06LS1C2 -> HYG025N06LS1C2NMOS; footprint easyeda2kicad:DFN-8_L5.9-W5.2-P1.27-LS6.2-BL -> (none)
- R10, R16, R17, R23, R24, R32, R33, R34, R9: footprint easyeda2kicad:R0805 -> (none)
- R11, R18, R25: value 47k -> 18k; footprint easyeda2kicad:R0805 -> (none)
- R12, R21, R28: value 36k -> 7k; footprint easyeda2kicad:R0805 -> (none)
- R13, R20, R27, R35: value 5k -> 1k; footprint easyeda2kicad:R0805 -> (none)
- R14: value 0 -> 6E-4; footprint easyeda2kicad:R0805 -> (none)
- R19, R26: footprint easyeda2kicad:RES-SMD_L6.4-W3.2_LRS2512 -> (none)
- R22, R29: value 220 -> 1k; footprint easyeda2kicad:R0805 -> (none)
- R30: value 5k -> 10k; footprint easyeda2kicad:R0805 -> (none)
- R31: value 47k -> 20k; footprint easyeda2kicad:R0805 -> (none)
- R36, R37, R38: value 220 -> 100; footprint easyeda2kicad:R0805 -> (none)
- ST-Link: renamed from ST-Link1; footprint Connector_PinHeader_2.54mm:PinHeader_2x04_P2.54mm_Vertical -> (none)
- TVS1: footprint easyeda2kicad:SOD-123FL_L2.7-W1.8-LS3.8-RD -> Diode_SMD:D_SMF
Connections:
- net +12V: now also 12V_SD1.3 (FB), C21.1, C29.1, C42.1, C45.1, L5.2
- net +3V3MCU: now also C17.1, C50.1, U8.5 (V+)
- net +ESC: now also 12V_SD1.1 (VIN), C43.1, C44.1
- net -3V3MCU: now also U13.8 (VSSA); no longer R14.1
- net -ESC: now also R14.2, 12V_SD1.4 (~{EN}), 12V_SD1.5 (GND), 12V_SD1.6 (GND), 12V_SD1.7 (GND), 12V_SD1.8 (GND), C17.2, C21.2, C29.2, C42.2, C43.2, C44.2, C45.2, C50.2, D16.2 (A), U8.4 (-); no longer Q4.3 (S), R18.2
- net A_Phase: now also D9.1
- net B_Phase: now also D11.1
- net C_Phase: now also D13.1
- net MCU_AI: now also C18.1, R15.2; no longer R29.2
- net MCU_CI: now also R29.2, C51.1; no longer C27.1, R22.2
- net at C25.2, R20.2, R21.1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: now also D11.2
- net at U9.2 (GND): now also C51.2
- net at C49.2, R27.2, R28.1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: now also D13.2
- net at C19.2, R12.1, R13.2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: now also D9.2
- net MCU_BI: now reaches U13.26 (PB13)
- net MCU_BI: now also C27.1, R22.2
- net Shunt_A: no longer names the net of Q2.3 (S), R11.2
- net Shunt_A: now also R14.1, U8.3 (+); no longer R26.1, U9.3 (+)
- net Shunt_C: no longer names the net of R19.1, U4.3 (+)
- net Shunt_C: now also Q4.3 (S), R18.2; no longer Q6.3 (S), R25.2
- removed net VSSA: R14.2, U13.8 (VSSA)
- new net: R15.1, U8.1
- new net: C18.2, U8.2 (GND)
- new net: Q6.3 (S), R25.2, R26.1, U9.3 (+)
- new net: 12V_SD1.2 (OUT), D16.1 (K), L5.1
- no-connect marks 22 -> 2
Other:
- note added: "ADC4_CH5"
- note added: "LEDs 5mA x 2"
- note added: "Max Drain Output: 4A Switching Time: 170nS Maximum Frequency: 5.88MHz"
- note added: "Max Voltage Drop: 0.03V Dissipation: 1.5W (7.13°)"
- note removed: "Drain Output (MAX): 4A Switching Time: 170nS Maximum Frequency: 5.88MHz"
- note removed: "LEDs 15mA x 2"
- note removed: "Phase Outputs"
- note removed: "Voltage Drop (MAX): 0.03V Dissipation: 1.5W (7.13°)"
- moved on the sheet: C20, C22, C25, D10, D17, Q3, Q4, R16, R17, R18, R20, R21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
